File: hardware/jardim.kicad_sch (KiCad schematic)
At the start: 67 parts, among them J1 DC_INPUT, J10 DHT22_AMB, J11 LIGHT_SENSOR_1, J12 LIGHT_SENSOR_2, J13 LEVEL_SENSOR_1, J14 LEVEL_SENSOR_2, J15 SOIL_HUMIDITY_SENSOR_1, J16 SOIL_HUMIDITY_SENSOR_2, J2 PUMP_1, J3 PUMP_2, J4 LIGHT_1, J5 LIGHT_2, J6 HEAT_2, J7 HEAT_2, J8 DS12B20_2, J9 DS18B20_1, Q1 IRLB8721, Q2 IRLB8721, Q3 IRLB8721, Q4 IRLB8721, Q5 IRLB8721, Q6 IRLB8721, U1 AM2302

Commit message: miniaturizando com grade menor
Parts:
- added SW1, SW2, SW3: SW_Push, Button_Switch_THT:SW_PUSH_6mm, symbol Switch:SW_Push
- added U2: DM-OLED096-636, oled:MODULE_DM-OLED096-636, symbol DM-OLED096-636:DM-OLED096-636
- C1: value 100uF -> 220uF
- J6: value HEAT_2 -> HEAT_1

Commit message: buzzer e textos
Parts:
- added BZ1: Buzzer, Buzzer_Beeper:Buzzer_12x9.5RM7.6, symbol Device:Buzzer
- added D5: 1N5822, Diode_THT:D_DO-201AD_P15.24mm_Horizontal, symbol Device:D_Schottky
- added Q7: FQP30N06L, Package_TO_SOT_THT:TO-220-3_Horizontal_TabDown, symbol Transistor_FET:Q_NMOS_GDS
- added R20: 220, Resistor_THT:R_Axial_DIN0207_L6.3mm_D2.5mm_P10.16mm_Horizontal, symbol Device:R
- added R21: 10k, Resistor_THT:R_Axial_DIN0207_L6.3mm_D2.5mm_P10.16mm_Horizontal, symbol Device:R
- added SW4: SW_SPST, TerminalBlock_Phoenix:TerminalBlock_Phoenix_MKDS-1,5-2-5.08_1x02_P5.08mm_Horizontal, symbol Switch:SW_SPST
- Q1, Q2, Q3, Q4, Q5, Q6: value IRLB8721 -> FQP30N06L
- R19: footprint Resistor_THT:R_Axial_DIN0207_L6.3mm_D2.5mm_P10.16mm_Horizontal -> Resistor_THT:R_Axial_DIN0207_L6.3mm_D2.5mm_P7.62mm_Horizontal
Connections:
- net +12V: now also BZ1.1 (+), D5.1 (K)
- net +24V: now also SW4.1 (A); no longer F1.1
- net GND: now also Q7.3 (S), R21.1
- net IO17: now also R20.2
- new net: F1.1, SW4.2 (B)
- new net: BZ1.2 (-), D5.2 (A), Q7.2 (D)
- new net: Q7.1 (G), R20.1, R21.2
Other:
- note added: "BUZZER_CIRCUIT"
- note added: "DHT22"
- moved on the sheet: C1, C2, J_IN3, J_IN4, J_IN5, J_IN6, J_OUT3, J_OUT4, J_OUT5, J_OUT6

Commit message: avisos de serigrafia
Other:
- moved on the sheet: R19, U1
Changed lines of the file:
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@@
 	)
 	(rectangle
-		(start 217.17 54.61)
-		(end 251.46 76.2)
+		(start 220.98 55.88)
+		(end 255.27 77.47)
 		(stroke
 			(width 0)
@@
 	(text "DHT22"
 		(exclude_from_sim no)
-		(at 246.634 61.468 0)
+		(at 250.444 62.738 0)
 		(effects
 			(font
@@
 	)
 	(junction
-		(at 238.76 67.31)
+		(at 242.57 68.58)
 		(diameter 0)
 		(color 0 0 0 0)
@@
 	(wire
 		(pts
-			(xy 220.98 67.31) (xy 219.71 67.31)
+			(xy 224.79 68.58) (xy 223.52 68.58)
 		)
 		(stroke
@@
 	(wire
 		(pts
-			(xy 219.71 67.31) (xy 219.71 68.58)
+			(xy 223.52 68.58) (xy 223.52 69.85)
 		)
 		(stroke
@@
 	(wire
 		(pts
-			(xy 238.76 62.23) (xy 238.76 67.31)
+			(xy 242.57 63.5) (xy 242.57 68.58)
 		)
 		(stroke
@@
 	(wire
 		(pts
-			(xy 228.6 74.93) (xy 243.84 74.93)
+			(xy 232.41 76.2) (xy 247.65 76.2)
 		)
 		(stroke
@@
 	(wire
 		(pts
-			(xy 236.22 67.31) (xy 238.76 67.31)
+			(xy 240.03 68.58) (xy 242.57 68.58)
 		)
 		(stroke
@@
 	(wire
 		(pts
-			(xy 238.76 67.31) (xy 243.84 67.31)
+			(xy 242.57 68.58) (xy 247.65 68.58)
 		)
 		(stroke
@@
 	)
 	(label "IO16"
-		(at 228.6 74.93 0)
+		(at 232.41 76.2 0)
 		(effects
 			(font
@@
 	(symbol
 		(lib_id "Sensor:AM2302")
-		(at 228.6 67.31 270)
+		(at 232.41 68.58 270)
 		(unit 1)
 		(body_style 1)
@@
 		(fields_autoplaced yes)
 		(property "Reference" "U1"
-			(at 228.6 57.15 90)
+			(at 232.41 58.42 90)
 			(show_name no)
 			(do_not_autoplace no)
@@
 		)
 		(property "Value" "AM2302"
-			(at 228.6 59.69 90)
+			(at 232.41 60.96 90)
 			(show_name no)
 			(do_not_autoplace no)
@@
 		)
 		(property "Footprint" "Sensor:ASAIR_AM2302_P2.54mm_Vertical"
-			(at 218.44 67.31 0)
+			(at 222.25 68.58 0)
 			(hide yes)
 			(show_name no)
@@
 		)
 		(property "Datasheet" "http://akizukidenshi.com/download/ds/aosong/AM2302.pdf"
-			(at 234.95 71.12 0)
+			(at 238.76 72.39 0)
 			(hide yes)
 			(show_name no)
@@
 		)
 		(property "Description" "3.3 to 5.0V, Temperature and humidity module,  DHT22, AM2302"
-			(at 228.6 67.31 0)
+			(at 232.41 68.58 0)
 			(hide yes)
 			(show_name no)
@@
 	(symbol
 		(lib_id "power:+5V")
-		(at 238.76 62.23 0)
+		(at 242.57 63.5 0)
 		(unit 1)
 		(body_style 1)
@@
 		(fields_autoplaced yes)
 		(property "Reference" "#PWR039"
-			(at 238.76 66.04 0)
+			(at 242.57 67.31 0)
 			(hide yes)
 			(show_name no)
@@
 		)
 		(property "Value" "+5V"
-			(at 238.76 57.15 0)
+			(at 242.57 58.42 0)
 			(show_name no)
 			(do_not_autoplace no)
@@
 		)
 		(property "Footprint" ""
-			(at 238.76 62.23 0)
+			(at 242.57 63.5 0)
 			(hide yes)
 			(show_name no)
@@
 		)
 		(property "Datasheet" ""
-			(at 238.76 62.23 0)
+			(at 242.57 63.5 0)
 			(hide yes)
 			(show_name no)
@@
 		)
 		(property "Description" "Power symbol creates a global label with name \"+5V\""
-			(at 238.76 62.23 0)
+			(at 242.57 63.5 0)
 			(hide yes)
 			(show_name no)
@@
 	(symbol
 		(lib_id "Device:R")
-		(at 243.84 71.12 0)
+		(at 247.65 72.39 0)
 		(unit 1)
 		(body_style 1)
@@
 		(fields_autoplaced yes)
 		(property "Reference" "R19"
-			(at 246.38 69.8499 0)
+			(at 250.19 71.1199 0)
 			(show_name no)
 			(do_not_autoplace no)
@@
 		)
 		(property "Value" "10k"
-			(at 246.38 72.3899 0)
+			(at 250.19 73.6599 0)
 			(show_name no)
 			(do_not_autoplace no)
@@
 		)
 		(property "Footprint" "Resistor_THT:R_Axial_DIN0207_L6.3mm_D2.5mm_P7.62mm_Horizontal"
-			(at 242.062 71.12 90)
+			(at 245.872 72.39 90)
 			(hide yes)
 			(show_name no)
@@
 		)
 		(property "Datasheet" ""
-			(at 243.84 71.12 0)
+			(at 247.65 72.39 0)
 			(hide yes)
 			(show_name no)
@@
 		)
 		(property "Description" "Resistor"
-			(at 243.84 71.12 0)
+			(at 247.65 72.39 0)
 			(hide yes)
 			(show_name no)
@@
 	(symbol
 		(lib_id "power:GND")
-		(at 219.71 68.58 0)
+		(at 223.52 69.85 0)
 		(unit 1)
 		(body_style 1)
@@
 		(fields_autoplaced yes)
 		(property "Reference" "#PWR038"
-			(at 219.71 74.93 0)
+			(at 223.52 76.2 0)
 			(hide yes)
 			(show_name no)
@@
 		)
 		(property "Value" "GND"
-			(at 219.71 73.66 0)
+			(at 223.52 74.93 0)
 			(show_name no)
 			(do_not_autoplace no)
@@
 		)
 		(property "Footprint" ""
-			(at 219.71 68.58 0)
+			(at 223.52 69.85 0)
 			(hide yes)
 			(show_name no)
@@
 		)
 		(property "Datasheet" ""
-			(at 219.71 68.58 0)
+			(at 223.52 69.85 0)
 			(hide yes)
 			(show_name no)
@@
 		)
 		(property "Description" "Power symbol creates a global label with name \"GND\" , ground"
-			(at 219.71 68.58 0)
+			(at 223.52 69.85 0)
 			(hide yes)
 			(show_name no)

Commit message: atribuindo gpio e furações com pad
Connections:
- net +5V: now also U2.2 (VCC_IN)
- net GND: now also SW1.2, SW2.2, SW3.2, U2.1 (GND)
- net IO1: now also SW3.1
- net IO10: now also R1.1
- net IO11: now also R6.1
- net IO12: now also R9.1
- net IO13: now also R12.1
- net IO14: now also R15.1
- net IO15: now also R18.1; no longer R15.1
- net IO16: now also R20.2; no longer R18.1, R19.2, U1.2 (SDA)
- net IO17: now also R19.2, U1.2 (SDA); no longer R20.2
- net IO18: now also J10.2 (Pin_2)
- net IO35: now also J9.2 (Pin_2)
- net IO36: now also J8.2 (Pin_2)
- net IO37: now also J13.1 (Pin_1)
- net IO38: now also J14.1 (Pin_1)
- net IO4: now also J15.3 (Pin_3); no longer R1.1
- net IO47: now also SW1.1
- net IO48: now also SW2.1
- net IO5: now also J15.2 (Pin_2); no longer R6.1
- net IO6: no longer R9.1
- net IO7: no longer R12.1
- net IO8: now also J11.2 (Pin_2), J12.2 (Pin_2), U2.4 (SDA)
- net IO9: now also J11.3 (Pin_3), J12.3 (Pin_3), U2.3 (SCL)

Commit message: refazendo os conectores de perifericos. atualmente luz 1 concluida
Parts:
- removed C3, C6: 100uF 25V, Capacitor_THT:CP_Radial_D6.3mm_P2.50mm, symbol Device:C_Polarized
- removed C4, C5: 100nF 50V, Capacitor_THT:C_Disc_D5.0mm_W2.5mm_P5.00mm, symbol Device:C
- removed D3: 1N5822, Diode_THT:D_DO-201AD_P15.24mm_Horizontal, symbol Device:D_Schottky
- removed D4, D8, D9: LED, LED_THT:LED_D5.0mm, symbol Device:LED
- removed J3: PUMP_2, TerminalBlock_Phoenix:TerminalBlock_Phoenix_MKDS-1,5-2-5.08_1x02_P5.08mm_Horizontal, symbol Connector_Generic:Conn_01x02
- removed Q2, Q3, Q4: FQP30N06L, Package_TO_SOT_THT:TO-220-3_Vertical, symbol Transistor_FET:IRLZ44N
- removed R10, R4, R7: 1k, Resistor_THT:R_Axial_DIN0207_L6.3mm_D2.5mm_P10.16mm_Horizontal, symbol Device:R
- removed R11, R5, R8: 10k, Resistor_THT:R_Axial_DIN0207_L6.3mm_D2.5mm_P10.16mm_Horizontal, symbol Device:R
- removed R12, R6, R9: 220, Resistor_THT:R_Axial_DIN0207_L6.3mm_D2.5mm_P10.16mm_Horizontal, symbol Device:R
- added D10, D12, D14, D6: 1N5822, Diode_THT:D_DO-201AD_P15.24mm_Horizontal, symbol Device:D_Schottky
- added D11, D13, D15: LED, LED_THT:LED_D5.0mm, symbol Device:LED
- added J17: PUMP_2, TerminalBlock_Phoenix:TerminalBlock_Phoenix_MKDS-1,5-2-5.08_1x02_P5.08mm_Horizontal, symbol Connector_Generic:Conn_01x02
- added Q3 (x2), Q8: FQP30N06L, Package_TO_SOT_THT:TO-220-3_Vertical, symbol Transistor_FET:IRLZ44N
- added R22, R7 (x2): 1k, Resistor_THT:R_Axial_DIN0207_L6.3mm_D2.5mm_P10.16mm_Horizontal, symbol Device:R
- added R23, R8 (x2): 10k, Resistor_THT:R_Axial_DIN0207_L6.3mm_D2.5mm_P10.16mm_Horizontal, symbol Device:R
- added R24, R9 (x2): 220, Resistor_THT:R_Axial_DIN0207_L6.3mm_D2.5mm_P10.16mm_Horizontal, symbol Device:R
- J4: value LIGHT_1 -> PUMP_2
- J5: value LIGHT_2 -> PUMP_2
- J6: value HEAT_1 -> PUMP_2
- J7: value HEAT_2 -> PUMP_2
- Q7: value FQP30N06L -> BC337; footprint Package_TO_SOT_THT:TO-220-3_Horizontal_TabDown -> Package_TO_SOT_THT:TO-92_Inline_Horizontal2
Connections:
- net +12V: now also J4.1 (Pin_1), J6.1 (Pin_1), J7.1 (Pin_1), R13.1, R16.1, R3.2, D10.1 (K), D12.1 (K), D14.1 (K), D6.1 (K), J17.1 (Pin_1), R22.1, R7.1; no longer R3.1
- net +24V: now also R7.1; no longer J4.1 (Pin_1), J6.1 (Pin_1), J7.1 (Pin_1), R13.1, R16.1
- net GND: now also Q3.3 (S), Q3.3 (S), Q8.3 (S), R23.1, R8.1, R8.1
- net IO11: now also R15.1, R18.1, R24.1, R9.1
- net IO12: now also R9.1
- net IO14: no longer R15.1
- net IO15: no longer R18.1
- net PUMP_1_SW_NEG: now reaches D1.2 (A), D2.1 (K), J2.2 (Pin_2), Q1.2 (D)
- net PUMP_2_SW_NEG: now reaches J6.2 (Pin_2), Q5.2 (D)
- net PUMP_2_SW_NEG: now also D7.1 (K), J4.2 (Pin_2), J7.2 (Pin_2), Q6.2 (D), D10.2 (A), D11.1 (K), D12.2 (A), D13.1 (K), D14.2 (A), D15.1 (K), D6.2 (A), J17.2 (Pin_2), Q3.2 (D), Q8.2 (D)
- net LIGHT_1_SW_NEG: now reaches J5.2 (Pin_2)
- net LIGHT_1_SW_NEG: now also D6.1 (K), Q3.2 (D); no longer D7.1 (K)
- net at D2.2 (A): now also R3.1; no longer R3.2
- net at R16.2: now also D13.2 (A)
- net at D6.2 (A): now also R7.2
- net at R13.2: now also D11.2 (A)
- net at D7.2 (A): now also R7.2
- new net: D15.2 (A), R22.2
- new net: Q3.1 (G), R8.2, R9.2 (x2)
- new net: Q8.1 (G), R23.2, R24.2
Other:
- note added: "BUTTONS"
- note added: "OLED"
- note removed: "HEAT_1"
- note removed: "HEAT_2"
- note removed: "LIGHT_2"
- moved on the sheet: BZ1, D1, D2, D5, J2, PH_1, PH_2, Q1, Q7, R1, R19, R2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

Commit message: corrigido todos os modulos perifericos
Parts:
- removed D10, D12, D14: 1N5822, Diode_THT:D_DO-201AD_P15.24mm_Horizontal, symbol Device:D_Schottky
- added H1, H2, H3, H4: MountingHole_Pad, MountingHole:MountingHole_3.2mm_M3_Pad_Via, symbol Mechanical:MountingHole_Pad
- J4: renamed from J5; value PUMP_2 -> LIGHT_1
- J5: renamed from J6; value PUMP_2 -> LIGHG_2
- J6: renamed from J7; value PUMP_2 -> HEAT_1
- J7: renamed from J17; value PUMP_2 -> HEAT_2
- renumbered D6 to D3, D7 to D4, D11 to D7, D13 to D8, D15 to D9, J4 to J3, Q3 to Q2, Q5 to Q4, Q6 to Q5, Q8 to Q6, R13 to R10, R14 to R11, R15 to R12, R16 to R13, R17 to R14, R18 to R15, R22 to R16, R23 to R17, R24 to R18, R7 to R4, R8 to R5, R9 to R6
Connections:
- net +12V: no longer J5.1 (Pin_1), J6.1 (Pin_1), J7.1 (Pin_1), R10.1, R13.1, R16.1
- net +24V: now also J5.1 (Pin_1), J6.1 (Pin_1), J7.1 (Pin_1), R10.1, R13.1, R16.1
- net GND: now also H1.1, H2.1, H3.1, H4.1
- net IO11: no longer R12.1, R15.1, R18.1
- net IO13: now also R12.1
- net IO14: now also R15.1
- net IO15: now also R18.1
- net PUMP_2_SW_NEG: no longer D7.1 (K), D8.1 (K), D9.1 (K), J5.2 (Pin_2), J6.2 (Pin_2), J7.2 (Pin_2), Q4.2 (D), Q5.2 (D), Q6.2 (D)
- new net HEATER_1_SW_NEG: D8.1 (K), J6.2 (Pin_2), Q5.2 (D)
- new net HEATER_2_SW_NEG: D9.1 (K), J7.2 (Pin_2), Q6.2 (D)
- new net LIGHT_2_SW_NEG: D7.1 (K), J5.2 (Pin_2), Q4.2 (D)
Other:
- note added: "HEATER_1"
- note added: "HEATER_2"
- note added: "LIGHT_2"
- moved on the sheet: BZ1, C1, C2, D1, D2, D3, D4, D5, D6, D7, D8, D9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

Commit message: to-do usb
Parts:
- added J17: USB_A, symbol Connector:USB_A
- added J18: USB_C_Receptacle_PowerOnly_6P, symbol Connector:USB_C_Receptacle_PowerOnly_6P
Connections:
- new net: J18.A12 (GND), J18.B12 (GND)
- new net: J18.A9 (VBUS), J18.B9 (VBUS)
Changed lines of the file:
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@@
 	)
 	(symbol
+		(lib_id "Connector:USB_A")
+		(at 62.23 220.98 0)
+		(unit 1)
+		(body_style 1)
+		(exclude_from_sim no)
+		(in_bom yes)
+		(on_board yes)
+		(in_pos_files yes)
+		(dnp no)
+		(fields_autoplaced yes)
+		(property "Reference" "J17"
+			(at 62.23 208.28 0)
+			(show_name no)
+			(do_not_autoplace no)
+			(effects
+				(font
+					(size 1.27 1.27)
+				)
+			)
+		)
+		(property "Value" "USB_A"
+			(at 62.23 210.82 0)
+			(show_name no)
+			(do_not_autoplace no)
+			(effects
+				(font
+					(size 1.27 1.27)
+				)
+			)
+		)
+		(property "Footprint" ""
+			(at 66.04 222.25 0)
+			(hide yes)
+			(show_name no)
+			(do_not_autoplace no)
+			(effects
+				(font
+					(size 1.27 1.27)
+				)
+			)
+		)
+		(property "Datasheet" ""
+			(at 66.04 222.25 0)
+			(hide yes)
+			(show_name no)
+			(do_not_autoplace no)
+			(effects
+				(font
+					(size 1.27 1.27)
+				)
+			)
+		)
+		(property "Description" "USB Type A connector"
+			(at 62.23 220.98 0)
+			(hide yes)
+			(show_name no)
+			(do_not_autoplace no)
+			(effects
+				(font
+					(size 1.27 1.27)
+				)
+			)
+		)
+		(pin "1"
+		)
+		(pin "2"
+		)
+		(pin "3"
+		)
+		(pin "4"
+		)
+		(pin "SH"
+		)
+		(instances
+			(project "jardim"
+				(path "/be2a7050-4dcf-40a5-a221-48a7948dc32a"
+					(reference "J17")
+					(unit 1)
+				)
+			)
+		)
+	)
+	(symbol
 		(lib_id "power:GND")
 		(at 345.44 113.03 0)
@@
 					(unit 1)
 				)
+			)
+		)
+	)
+	(symbol
+		(lib_id "Connector:USB_C_Receptacle_PowerOnly_6P")
+		(at 92.71 226.06 0)
+		(unit 1)
+		(body_style 1)
+		(exclude_from_sim no)
+		(in_bom yes)
+		(on_board yes)
+		(in_pos_files yes)
+		(dnp no)
+		(fields_autoplaced yes)
+		(property "Reference" "J18"
+			(at 92.71 208.28 0)
+			(show_name no)
+			(do_not_autoplace no)
+			(effects
+				(font
+					(size 1.27 1.27)
+				)
+			)
+		)
+		(property "Value" "USB_C_Receptacle_PowerOnly_6P"
+			(at 92.71 210.82 0)
+			(show_name no)
+			(do_not_autoplace no)
+			(effects
+				(font
+					(size 1.27 1.27)
+				)
+			)
+		)
+		(property "Footprint" ""
+			(at 96.52 223.52 0)
+			(hide yes)
+			(show_name no)
+			(do_not_autoplace no)
+			(effects
+				(font
+					(size 1.27 1.27)
+				)
+			)
+		)
+		(property "Datasheet" "https://www.usb.org/sites/default/files/documents/usb_type-c.zip"
+			(at 92.71 226.06 0)
+			(hide yes)
+			(show_name no)
+			(do_not_autoplace no)
+			(effects
+				(font
+					(size 1.27 1.27)
+				)
+			)
+		)
+		(property "Description" "USB Power-Only 6P Type-C Receptacle connector"
+			(at 92.71 226.06 0)
+			(hide yes)
+			(show_name no)
+			(do_not_autoplace no)
+			(effects
+				(font
+					(size 1.27 1.27)
+				)
+			)
+		)
+		(pin "B12"
+		)
+		(pin "A9"
+		)
+		(pin "A5"
+		)
+		(pin "B9"
+		)
+		(pin "SH"
+		)
+		(pin "A12"
+		)
+		(pin "B5"
+		)
+		(instances
+			(project "jardim"
+				(path "/be2a7050-4dcf-40a5-a221-48a7948dc32a"
+					(reference "J18")
+					(unit 1)
+				)
